Commit message: aliengo; reuse classic TG; DynamicsInfo; fix plotter; reset LinearVelocityReward; better main

File: urdf/aliengo/urdf/aliengo.urdf (robot description, URDF)
Before this commit: robot aliengo_description, 25 links, 24 joints
Links:
- removed link camera_depth_frame
- removed link camera_depth_optical_frame
- removed link camera_link
- removed link camera_rgb_frame
- removed link camera_rgb_optical_frame
- removed link hokuyo_frame
- link FL_calf: geometry collision box size=0.25 0.0208 0.016; visual mesh filename=../meshes/calf.stl scale=1 1 1
- link FL_hip: geometry collision cylinder length=0.0418 radius=0.046; visual mesh filename=../meshes/hip.stl scale=1 1 1
- link FL_thigh: geometry collision box size=0.25 0.0374 0.043; visual mesh filename=../meshes/thigh.stl scale=1 1 1
- link FR_calf: geometry collision box size=0.25 0.0208 0.016; visual mesh filename=../meshes/calf.stl scale=1 1 1
- link FR_hip: geometry collision cylinder length=0.0418 radius=0.046; visual mesh filename=../meshes/hip.stl scale=1 1 1
- link FR_thigh: geometry collision box size=0.25 0.0374 0.043; visual mesh filename=../meshes/thigh_mirror.stl scale=1 1 1
- link RL_calf: geometry collision box size=0.25 0.0208 0.016; visual mesh filename=../meshes/calf.stl scale=1 1 1
- link RL_hip: geometry collision cylinder length=0.0418 radius=0.046; visual mesh filename=../meshes/hip.stl scale=1 1 1
- link RL_thigh: geometry collision box size=0.25 0.0374 0.043; visual mesh filename=../meshes/thigh.stl scale=1 1 1
- link RR_calf: geometry collision box size=0.25 0.0208 0.016; visual mesh filename=../meshes/calf.stl scale=1 1 1
- link RR_hip: geometry collision cylinder length=0.0418 radius=0.046; visual mesh filename=../meshes/hip.stl scale=1 1 1
- link RR_thigh: geometry collision box size=0.25 0.0374 0.043; visual mesh filename=../meshes/thigh_mirror.stl scale=1 1 1
- link base: mass None -> 0.001
- link imu_link: geometry collision box size=.001 .001 .001; visual box size=0.001 0.001 0.001
- link trunk: geometry collision box size=0.647 0.15 0.112; visual mesh filename=../meshes/trunk.stl scale=1 1 1
Joints:
- removed joint camera_depth_joint
- removed joint camera_depth_optical_joint
- removed joint camera_joint
- removed joint camera_rgb_joint
- removed joint camera_rgb_optical_joint
- removed joint hokuyo_joint
- joint FL_calf_joint: limit lower=-2.77507351067 upper=-0.645771823238 effort=55 velocity=16 -> lower=-2.77507351067 upper=-0.645771823238 effort=44.4 velocity=40
- joint FL_hip_joint: limit lower=-1.2217304764 upper=1.2217304764 effort=44 velocity=20 -> lower=-1.2217304764 upper=1.2217304764 effort=44.4 velocity=40
- joint FL_thigh_joint: limit effort=44 velocity=20 -> effort=44.4 velocity=40
- joint FR_calf_joint: limit lower=-2.77507351067 upper=-0.645771823238 effort=55 velocity=16 -> lower=-2.77507351067 upper=-0.645771823238 effort=44.4 velocity=40
- joint FR_hip_joint: limit lower=-1.2217304764 upper=1.2217304764 effort=44 velocity=20 -> lower=-1.2217304764 upper=1.2217304764 effort=44.4 velocity=40
- joint FR_thigh_joint: limit effort=44 velocity=20 -> effort=44.4 velocity=40
- joint RL_calf_joint: limit lower=-2.77507351067 upper=-0.645771823238 effort=55 velocity=16 -> lower=-2.77507351067 upper=-0.645771823238 effort=44.4 velocity=40
- joint RL_hip_joint: limit lower=-1.2217304764 upper=1.2217304764 effort=44 velocity=20 -> lower=-1.2217304764 upper=1.2217304764 effort=44.4 velocity=40
- joint RL_thigh_joint: limit effort=44 velocity=20 -> effort=44.4 velocity=40
- joint RR_calf_joint: limit lower=-2.77507351067 upper=-0.645771823238 effort=55 velocity=16 -> lower=-2.77507351067 upper=-0.645771823238 effort=44.4 velocity=40
- joint RR_hip_joint: limit lower=-1.2217304764 upper=1.2217304764 effort=44 velocity=20 -> lower=-1.2217304764 upper=1.2217304764 effort=44.4 velocity=40
- joint RR_thigh_joint: limit effort=44 velocity=20 -> effort=44.4 velocity=40
- joint imu_joint: origin (none) -> xyz=0 0 0 rpy=0 0 0

Commit message: aliengo

File: urdf/aliengo/urdf/aliengo.urdf (robot description, URDF)
Before this commit: robot aliengo_description, 25 links, 24 joints
Links:
- removed link camera_depth_frame
- removed link camera_depth_optical_frame
- removed link camera_link
- removed link camera_rgb_frame
- removed link camera_rgb_optical_frame
- removed link hokuyo_frame
- link FL_calf: geometry collision box size=0.25 0.0208 0.016; visual mesh filename=../meshes/calf.stl scale=1 1 1
- link FL_hip: geometry collision cylinder length=0.0418 radius=0.046; visual mesh filename=../meshes/hip.stl scale=1 1 1
- link FL_thigh: geometry collision box size=0.25 0.0374 0.043; visual mesh filename=../meshes/thigh.stl scale=1 1 1
- link FR_calf: geometry collision box size=0.25 0.0208 0.016; visual mesh filename=../meshes/calf.stl scale=1 1 1
- link FR_hip: geometry collision cylinder length=0.0418 radius=0.046; visual mesh filename=../meshes/hip.stl scale=1 1 1
- link FR_thigh: geometry collision box size=0.25 0.0374 0.043; visual mesh filename=../meshes/thigh_mirror.stl scale=1 1 1
- link RL_calf: geometry collision box size=0.25 0.0208 0.016; visual mesh filename=../meshes/calf.stl scale=1 1 1
- link RL_hip: geometry collision cylinder length=0.0418 radius=0.046; visual mesh filename=../meshes/hip.stl scale=1 1 1
- link RL_thigh: geometry collision box size=0.25 0.0374 0.043; visual mesh filename=../meshes/thigh.stl scale=1 1 1
- link RR_calf: geometry collision box size=0.25 0.0208 0.016; visual mesh filename=../meshes/calf.stl scale=1 1 1
- link RR_hip: geometry collision cylinder length=0.0418 radius=0.046; visual mesh filename=../meshes/hip.stl scale=1 1 1
- link RR_thigh: geometry collision box size=0.25 0.0374 0.043; visual mesh filename=../meshes/thigh_mirror.stl scale=1 1 1
- link imu_link: geometry collision box size=.001 .001 .001; visual box size=0.001 0.001 0.001
- link trunk: geometry collision box size=0.647 0.15 0.112; visual mesh filename=../meshes/trunk.stl scale=1 1 1
Joints:
- removed joint camera_depth_joint
- removed joint camera_depth_optical_joint
- removed joint camera_joint
- removed joint camera_rgb_joint
- removed joint camera_rgb_optical_joint
- removed joint hokuyo_joint
- joint FL_calf_joint: limit lower=-2.77507351067 upper=-0.645771823238 effort=55 velocity=16 -> lower=-2.77507351067 upper=-0.645771823238 effort=44.4 velocity=40
- joint FL_hip_joint: limit lower=-1.2217304764 upper=1.2217304764 effort=44 velocity=20 -> lower=-1.2217304764 upper=1.2217304764 effort=44.4 velocity=40
- joint FL_thigh_joint: limit effort=44 velocity=20 -> effort=44.4 velocity=40
- joint FR_calf_joint: limit lower=-2.77507351067 upper=-0.645771823238 effort=55 velocity=16 -> lower=-2.77507351067 upper=-0.645771823238 effort=44.4 velocity=40
- joint FR_hip_joint: limit lower=-1.2217304764 upper=1.2217304764 effort=44 velocity=20 -> lower=-1.2217304764 upper=1.2217304764 effort=44.4 velocity=40
- joint FR_thigh_joint: limit effort=44 velocity=20 -> effort=44.4 velocity=40
- joint RL_calf_joint: limit lower=-2.77507351067 upper=-0.645771823238 effort=55 velocity=16 -> lower=-2.77507351067 upper=-0.645771823238 effort=44.4 velocity=40
- joint RL_hip_joint: limit lower=-1.2217304764 upper=1.2217304764 effort=44 velocity=20 -> lower=-1.2217304764 upper=1.2217304764 effort=44.4 velocity=40
- joint RL_thigh_joint: limit effort=44 velocity=20 -> effort=44.4 velocity=40
- joint RR_calf_joint: limit lower=-2.77507351067 upper=-0.645771823238 effort=55 velocity=16 -> lower=-2.77507351067 upper=-0.645771823238 effort=44.4 velocity=40
- joint RR_hip_joint: limit lower=-1.2217304764 upper=1.2217304764 effort=44 velocity=20 -> lower=-1.2217304764 upper=1.2217304764 effort=44.4 velocity=40
- joint RR_thigh_joint: limit effort=44 velocity=20 -> effort=44.4 velocity=40
- joint imu_joint: origin (none) -> xyz=0 0 0 rpy=0 0 0

Commit message: fix tg for aliengo

File: urdf/aliengo/urdf/aliengo.urdf (robot description, URDF)
Before this commit: robot aliengo_description, 19 links, 18 joints
Links:
- link base: mass None -> 0.001
